File: PCB/PCB.kicad_sch (KiCad schematic)
At the start: 111 parts, among them J1 External Trig, J3 Conn_Coaxial, J4 RJ12, J5 Programming Header, J6 Camera TRS, J7 Conn_Coaxial, J8 USB_C_Receptacle_USB2.0_14P, Q3 MMBF170, Q4 MMBF170, Q5 FDN340P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

Commit message: Rev 2 of the PCB with modified test firmware and enclosure
Parts:
- removed C15, C16: 10nF, Capacitor_SMD:C_0805_2012Metric, symbol Device:C
- removed D2: ESDA14V2SC5, Package_TO_SOT_SMD:SOT-23-5, symbol Power_Protection:ESDA14V2SC5
- removed J3, J7: Conn_Coaxial, Connector_Coaxial:BNC_TEConnectivity_1478035_Horizontal, symbol Connector:Conn_Coaxial
- removed L1: 1uH, Inductor_SMD:L_1206_3216Metric, symbol Device:L
- removed Q5: FDN340P, Package_TO_SOT_SMD:SOT-23, symbol Transistor_FET:FDN340P
- removed Q6: MMBF170, Package_TO_SOT_SMD:SOT-23, symbol Transistor_FET:MMBF170
- removed R11, R12: 100k, Resistor_SMD:R_0805_2012Metric, symbol Device:R
- removed R15: 56k, Resistor_SMD:R_0805_2012Metric, symbol Device:R
- removed R20, R54: 10k, Resistor_SMD:R_0805_2012Metric, symbol Device:R
- removed R3, R4, R46: 1k, Resistor_SMD:R_0805_2012Metric, symbol Device:R
- removed R47: 0, Resistor_SMD:R_0805_2012Metric, symbol Device:R
- removed U1: TPS631000, Package_TO_SOT_SMD:SOT-583-8, symbol ProjectSymbols:TPS631000
- removed U7: STM32G071K8Tx, Package_QFP:LQFP-32_7x7mm_P0.8mm, symbol MCU_ST_STM32G0:STM32G071K8Tx
- added J2: Conn_01x02_Socket, Connector_PinHeader_2.54mm:PinHeader_1x02_P2.54mm_Vertical, symbol Connector:Conn_01x02_Socket
- added R42: 1k, Resistor_SMD:R_0805_2012Metric, symbol Device:R
- added U1: STM32G071K8Tx, Package_QFP:LQFP-32_7x7mm_P0.8mm, symbol MCU_ST_STM32G0:STM32G071K8Tx
- added U9: TLV75733PDBV, Package_TO_SOT_SMD:SOT-23-5, symbol Regulator_Linear:TLV75733PDBV
- C13: value 47uF -> 10uF
- C4: value 22uF -> 10uF
- R24: value 10k -> 0; now not fitted
- R25: value 10k -> 1k
- TP1: footprint TestPoint:TestPoint_Keystone_5005-5009_Compact -> TestPoint:TestPoint_Pad_D1.5mm
Connections:
- net +3.3V: now also U1.4 (VDD), U9.5 (OUT); no longer R35.2, R37.2
- net 3V3_EN: now also U9.3 (EN)
- net 3V3_EN_MCU: now also U1.19 (PA9/UCPD1_DBCC1)
- net AUDIO_DEC: now also U1.10 (PA3)
- net BATT-OUT: now also R42.1, U9.1 (IN)
- net BT1: now also R6.2, SW1.1, U1.11 (PA4)
- net BT2: now also R7.2, SW2.1, U1.12 (PA5)
- net CAM_FOC: now also U1.9 (PA2)
- net CAM_TRG: now also U1.14 (PA7)
- net CLK: now also U1.32 (PB8)
- net EXT_TRIG_IN: now also U1.7 (PA0)
- net EXT_UART_RX: now also U1.15 (PB0)
- net EXT_UART_TX: now also U1.17 (PB2)
- net GND: now also R35.1, R37.1, J2.2 (Pin_2), U1.5 (VSS), U9.2 (GND)
- net LCD_BLK: now also U1.26 (PA15)
- net LCD_CS: now also U1.28 (PB4)
- net LCD_DC: now also U1.29 (PB5)
- net LCD_RES: now also U1.30 (PB6)
- net LIGHT_DEC: now also U1.8 (PA1)
- net MOSI: now also U1.31 (PB7)
- net PROG_RST: now also U1.6 (PF2)
- net PROG_SWCLK: now also U1.25 (PA14)
- net PROG_SWDIO: now also U1.24 (PA13)
- net ROT_A: now also U1.18 (PA8)
- net ROT_B: now also U1.22 (PA9/PA11)
- net ROT_S: now also U1.16 (PB1)
- net TIA_SEL1: now also U1.23 (PA10/PA12)
- net TIA_SEL2: now also U1.21 (PA10/UCPD1_DBCC2)
- net TRG_{OUT}_{1}: now also J2.1 (Pin_1)
- net TRIG_{1}: now also U1.13 (PA6)
- net ~{CHR}: now also U1.3 (PC15)
- net ~{PGOOD}: now also U1.2 (PC14)
- net at C2.1, D1.1 (K), TP2.1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: now also U5.2 (-); no longer U5.3 (+)
- net at Q4.1 (G), R36.2: now also R37.2; no longer R37.1
- net at C3.2, R8.2, R9.2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: now also U5.3 (+); no longer U5.2 (-)
- net at C11.2, R14.2, R19.2: now also U5.5 (+); no longer U5.6 (-)
- net at Q3.1 (G), R34.2: now also R35.2; no longer R35.1
- net at C1.1, C8.2, R10.2: now also U5.6 (-); no longer U5.5 (+)
- net BATT-EN1: no longer names the net of R24.1, U4.6 (EN1)
- net BATT-EN1: now also R42.2
- net BATT-EN2: no longer names the net of R25.1, U4.5 (EN2)
- net CC1: no longer names the net of J8.A5 (CC1), R18.1
- net CC2: no longer names the net of J8.B5 (CC2), R17.1
- no-connect marks 6 -> 9
Other:
- note removed: "Battery Monitor"
- moved on the sheet: BT2, C13, C17, C4, C5, C7, J1, Q3, R21, R22, R23, R25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
